File: ESP-Switch.kicad_pcb (KiCad board)
At the start: 2 copper layers, 119.3 x 58.4 mm, 46 parts, among them K1 Relay, K2 Relay, K3 Relay, K4 Relay, Q1 BC817, Q2 BC817, Q3 BC817, Q4 BC817, U1 AMS1117-3.3

Commit message: WIP
Parts:
- removed the H1 at (107.1, 79.1)
- removed the H1 at (154.3, 27.8)
- added H1: MountingHole, MountingHole:MountingHole_3.2mm_M3_DIN965, F.Cu at (43.0, 78.3)
- added H2: MountingHole, MountingHole:MountingHole_3.2mm_M3_DIN965, F.Cu at (61.7, 79.2)
- H3, H4: footprint MountingHole:MountingHole_2.2mm_M2_ISO7380_Pad_TopBottom -> MountingHole:MountingHole_3.2mm_M3_DIN965
- PS1: renamed from Power Supply
- ROP1, ROP2, ROP3, ROP4: value 470R -> 1K
- RQ1, RQ2, RQ3, RQ4: value 120R -> 1K
- moved H4 65.0 mm to (107.5, 79.2)
- moved H3 57.9 mm to (66.7, 79.2)
- renumbered Mains to J1, A to LED1, B to LED2, C to LED3, D to LED4, ON to PWR1, ESP-01 to U2
Other:
- outline, holes or cut-outs redrawn
