File: ESP-Switch.sch (KiCad schematic (older format))
At the start: 46 parts, among them J1 AC/In, K1 Relay, K2 Relay, K3 Relay, K4 Relay, Q1 BC817, Q2 BC817, Q3 BC817, Q4 BC817, U1 AMS1117-3.3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

Commit message: WIP
Parts:
- H1, H2, H3, H4: footprint MountingHole:MountingHole_2.2mm_M2_ISO7380_Pad_TopBottom -> MountingHole:MountingHole_3.2mm_M3_DIN965
Changed lines of the file:
@@
 F 0 "H4" H 14065 2476 50  0000 L CNN
 F 1 "MountingHole" H 14065 2385 50  0000 L CNN
-F 2 "MountingHole:MountingHole_2.2mm_M2_ISO7380_Pad_TopBottom" H 13965 2430 50  0001 C CNN
+F 2 "MountingHole:MountingHole_3.2mm_M3_DIN965" H 13965 2430 50  0001 C CNN
 F 3 "~" H 13965 2430 50  0001 C CNN
 	1    13965 2430
@@
 F 0 "H1" H 14050 2736 50  0000 L CNN
 F 1 "MountingHole" H 14050 2645 50  0000 L CNN
-F 2 "MountingHole:MountingHole_2.2mm_M2_ISO7380_Pad_TopBottom" H 13950 2690 50  0001 C CNN
+F 2 "MountingHole:MountingHole_3.2mm_M3_DIN965" H 13950 2690 50  0001 C CNN
 F 3 "~" H 13950 2690 50  0001 C CNN
 	1    13950 2690
@@
 F 0 "H3" H 14055 3001 50  0000 L CNN
 F 1 "MountingHole" H 14055 2910 50  0000 L CNN
-F 2 "MountingHole:MountingHole_2.2mm_M2_ISO7380_Pad_TopBottom" H 13955 2955 50  0001 C CNN
+F 2 "MountingHole:MountingHole_3.2mm_M3_DIN965" H 13955 2955 50  0001 C CNN
 F 3 "~" H 13955 2955 50  0001 C CNN
 	1    13955 2955
@@
 F 0 "H2" H 14050 3276 50  0000 L CNN
 F 1 "MountingHole" H 14050 3185 50  0000 L CNN
-F 2 "MountingHole:MountingHole_2.2mm_M2_ISO7380_Pad_TopBottom" H 13950 3230 50  0001 C CNN
+F 2 "MountingHole:MountingHole_3.2mm_M3_DIN965" H 13950 3230 50  0001 C CNN
 F 3 "~" H 13950 3230 50  0001 C CNN
 	1    13950 3230
